File: ZIN70 Nixie Clock.kicad_pcb (KiCad board)
At the start: 2 copper layers, 270 x 90 mm, 61 parts, among them Q1 PN2222A, Q2 PN2222A, Q3 PN2222A, Q4 PN2222A, U1 HV5122, U2 HV5122, U3 OKI-78SR-3.3_1.5-W36-C, U4 OKI-78SR-3.3_1.5-W36-C

Commit message: Adjustments I forgot to save
Other:
- board text removed: "Only batteries or plug! Not both!"
